File: hardware/masterUnit_kiCad/master_unit.kicad_pcb (KiCad board)
At the start: 2 copper layers, 62.2 x 141 mm, 13 parts, among them IC1 THVD8000DDFR, J1 Conn_01x03, J2 Conn_01x02, U1 DEV-15583

Commit message: updated pcb layout with new LED
Parts:
- added D1: LED_blue, LED_SMD:LED_1206_3216Metric, F.Cu at (90.2, 160.1)
- added D2: LED_green, LED_SMD:LED_1206_3216Metric, F.Cu at (117.6, 162.4)
- added D3: LED_red, LED_SMD:LED_1206_3216Metric, F.Cu at (117.5, 157.2)
- added R3: 1k, Resistor_SMD:R_1206_3216Metric, F.Cu at (93.1, 157.5)
- added R4: 1k, Resistor_SMD:R_1206_3216Metric, F.Cu at (112.0, 162.4)
- added R5: 1k, Resistor_SMD:R_1206_3216Metric, F.Cu at (112.1, 157.2)
Routing:
- net Net-(IC1-Pad1): track 23.5 -> 36.2 mm, vias 0 -> 2
- net GND: track 26.3 -> 34.1 mm, vias 2 -> 4
- net Net-(IC1-Pad4): track 34.0 -> 39.2 mm
- net 3.3V: track 40.9 -> 44.1 mm
- net Net-(D2-Pad2): track 0.00 -> 2.73 mm
- net Net-(D1-Pad2): track 0.00 -> 2.69 mm
- net Net-(D3-Pad2): track 0.00 -> 2.47 mm
Other:
- board text added: "Power"
- board text added: "Rx"
- board text added: "Tx"
